Commit message: mujoco testing file

File: dev/scripts/urdf/ur_description/mujoco_test/ur20.urdf (robot description, URDF)
Before this commit: robot ur20_robot, 11 links, 10 joints
Links:
- link base_link_inertia: geometry collision mesh filename=meshes/ur20/collision/base.stl; visual mesh filename=meshes/ur20/visual/base.dae
- link forearm_link: geometry collision mesh filename=meshes/ur20/collision/forearm.stl; visual mesh filename=meshes/ur20/visual/forearm.dae
- link shoulder_link: geometry collision mesh filename=meshes/ur20/collision/shoulder.stl; visual mesh filename=meshes/ur20/visual/shoulder.dae
- link upper_arm_link: geometry collision mesh filename=meshes/ur20/collision/upperarm.stl; visual mesh filename=meshes/ur20/visual/upperarm.dae
- link wrist_1_link: geometry collision mesh filename=meshes/ur20/collision/wrist1.stl; visual mesh filename=meshes/ur20/visual/wrist1.dae
- link wrist_2_link: geometry collision mesh filename=meshes/ur20/collision/wrist2.stl; visual mesh filename=meshes/ur20/visual/wrist2.dae
- link wrist_3_link: geometry collision mesh filename=meshes/ur20/collision/wrist3.stl; visual mesh filename=meshes/ur20/visual/wrist3.dae
